File: hardware/rev-d/kicad/link-commander.kicad_pcb (KiCad board)
At the start: 2 copper layers, 140 x 80 mm, 56 parts, among them J1 5V INPUT / GND, J2 USB 1, J3 USB 2, J4 KBD SDS-70J, J5 MOUSE SDS-70J, M1 RP2040-Zero SOCKETS, Q1 2N3904, Q2 2N3904, Q3 2N3904, Q4 2N3904, U1 TPS2042P, U2 CD4050BE

Commit message: Add through-hole test access and student probe guide to Rev D
Parts:
- added TP1: 5V_BOARD, LinkCommander:TestPoint_THT_1mm, F.Cu at (123.0, 48.0)
- added TP10: KBD_CLOCK, LinkCommander:TestPoint_THT_1mm, F.Cu at (56.0, 79.0)
- added TP11: MOUSE_DATA, LinkCommander:TestPoint_THT_1mm, F.Cu at (94.0, 81.0)
- added TP12: MOUSE_CLOCK, LinkCommander:TestPoint_THT_1mm, F.Cu at (126.0, 73.0)
- added TP13: GP8, LinkCommander:TestPoint_THT_1mm, F.Cu at (21.0, 57.0)
- added TP14: GP10, LinkCommander:TestPoint_THT_1mm, F.Cu at (53.0, 57.0)
- added TP15: GP12, LinkCommander:TestPoint_THT_1mm, F.Cu at (85.0, 57.0)
- added TP16: GP14, LinkCommander:TestPoint_THT_1mm, F.Cu at (117.0, 57.0)
- added TP17: GP9, LinkCommander:TestPoint_THT_1mm, F.Cu at (33.0, 57.0)
- added TP18: GP11, LinkCommander:TestPoint_THT_1mm, F.Cu at (65.0, 57.0)
- added TP19: GP13, LinkCommander:TestPoint_THT_1mm, F.Cu at (94.0, 55.0)
- added TP2: 5V_MODULE, LinkCommander:TestPoint_THT_1mm, F.Cu at (89.0, 44.0)
- added TP20: GP15, LinkCommander:TestPoint_THT_1mm, F.Cu at (129.0, 57.0)
- added TP21: USB1_FAULT, LinkCommander:TestPoint_THT_1mm, F.Cu at (42.0, 43.0)
- added TP22: USB2_FAULT, LinkCommander:TestPoint_THT_1mm, F.Cu at (58.0, 43.0)
- added TP23: GND, LinkCommander:TestPoint_THT_1mm, F.Cu at (15.0, 43.0)
- added TP24: GND, LinkCommander:TestPoint_THT_1mm, F.Cu at (76.0, 46.0)
- added TP25: GND, LinkCommander:TestPoint_THT_1mm, F.Cu at (61.0, 84.0)
- added TP26: GND, LinkCommander:TestPoint_THT_1mm, F.Cu at (140.0, 76.0)
- added TP3: 3V3, LinkCommander:TestPoint_THT_1mm, F.Cu at (93.0, 49.0)
- added TP4: USB1_5V, LinkCommander:TestPoint_THT_1mm, F.Cu at (47.0, 33.0)
- added TP5: USB2_5V, LinkCommander:TestPoint_THT_1mm, F.Cu at (60.0, 33.0)
- added TP6: KBD_5V, LinkCommander:TestPoint_THT_1mm, F.Cu at (23.0, 75.0)
- added TP7: MOUSE_5V, LinkCommander:TestPoint_THT_1mm, F.Cu at (94.0, 75.0)
- added TP8: 5V_INPUT, LinkCommander:TestPoint_THT_1mm, F.Cu at (145.0, 30.0)
- added TP9: KBD_DATA, LinkCommander:TestPoint_THT_1mm, F.Cu at (56.0, 73.0)
Routing:
- net GP9: track 10.9 -> 77.7 mm
- net GP11: track 18.1 -> 52.4 mm
- net 5V_BOARD: track 205.3 -> 171.9 mm
- net KBD_CLOCK: track 76.5 -> 106.6 mm, vias 1 -> 0
- net GND: track 423.7 -> 453.1 mm
- net GP14: track 45.7 -> 70.8 mm, vias 0 -> 1
- net GP15: track 38.4 -> 61.6 mm
- net MOUSE_DATA: track 51.4 -> 71.0 mm, vias 1 -> 0
- net 5V_MODULE: track 61.2 -> 79.2 mm
- net 5V_INPUT: track 28.1 -> 42.6 mm
- net USB1_5V: track 34.6 -> 45.3 mm
- net USB2_FAULT: track 43.7 -> 54.2 mm
- net GP13: track 25.4 -> 34.1 mm
- net KBD_DATA: track 105.2 -> 111.4 mm
- net USB2_5V: track 61.5 -> 67.7 mm
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Other:
- board text added: "GND"
- board text added: "USB1 D+"
- board text added: "USB1 D-"
- board text added: "USB2 D+"
- board text added: "USB2 D-"
