File: hardware/rev-d/kicad/link-commander.kicad_sch (KiCad schematic)
At the start: 50 parts, among them J1 5V INPUT / GND, J2 USB 1, J3 USB 2, J4 KBD SDS-70J, J5 MOUSE SDS-70J, M1 RP2040-Zero SOCKETS, Q1 2N3904, Q2 2N3904, Q3 2N3904, Q4 2N3904, U1 TPS2042P, U2 CD4050BE

Commit message: Add through-hole test access and student probe guide to Rev D
Parts:
- added TP1: 5V_BOARD, LinkCommander:TestPoint_THT_1mm, symbol LC_TP1
- added TP10: KBD_CLOCK, LinkCommander:TestPoint_THT_1mm, symbol LC_TP10
- added TP11: MOUSE_DATA, LinkCommander:TestPoint_THT_1mm, symbol LC_TP11
- added TP12: MOUSE_CLOCK, LinkCommander:TestPoint_THT_1mm, symbol LC_TP12
- added TP13: GP8, LinkCommander:TestPoint_THT_1mm, symbol LC_TP13
- added TP14: GP10, LinkCommander:TestPoint_THT_1mm, symbol LC_TP14
- added TP15: GP12, LinkCommander:TestPoint_THT_1mm, symbol LC_TP15
- added TP16: GP14, LinkCommander:TestPoint_THT_1mm, symbol LC_TP16
- added TP17: GP9, LinkCommander:TestPoint_THT_1mm, symbol LC_TP17
- added TP18: GP11, LinkCommander:TestPoint_THT_1mm, symbol LC_TP18
- added TP19: GP13, LinkCommander:TestPoint_THT_1mm, symbol LC_TP19
- added TP2: 5V_MODULE, LinkCommander:TestPoint_THT_1mm, symbol LC_TP2
- added TP20: GP15, LinkCommander:TestPoint_THT_1mm, symbol LC_TP20
- added TP21: USB1_FAULT, LinkCommander:TestPoint_THT_1mm, symbol LC_TP21
- added TP22: USB2_FAULT, LinkCommander:TestPoint_THT_1mm, symbol LC_TP22
- added TP23: GND, LinkCommander:TestPoint_THT_1mm, symbol LC_TP23
- added TP24: GND, LinkCommander:TestPoint_THT_1mm, symbol LC_TP24
- added TP25: GND, LinkCommander:TestPoint_THT_1mm, symbol LC_TP25
- added TP26: GND, LinkCommander:TestPoint_THT_1mm, symbol LC_TP26
- added TP3: 3V3, LinkCommander:TestPoint_THT_1mm, symbol LC_TP3
- added TP4: USB1_5V, LinkCommander:TestPoint_THT_1mm, symbol LC_TP4
- added TP5: USB2_5V, LinkCommander:TestPoint_THT_1mm, symbol LC_TP5
- added TP6: KBD_5V, LinkCommander:TestPoint_THT_1mm, symbol LC_TP6
- added TP7: MOUSE_5V, LinkCommander:TestPoint_THT_1mm, symbol LC_TP7
- added TP8: 5V_INPUT, LinkCommander:TestPoint_THT_1mm, symbol LC_TP8
- added TP9: KBD_DATA, LinkCommander:TestPoint_THT_1mm, symbol LC_TP9
Connections:
- net 3V3: now also TP3.1 (TEST)
- net 5V_BOARD: now also TP1.1 (TEST)
- net 5V_INPUT: now also TP8.1 (TEST)
- net 5V_MODULE: now also TP2.1 (TEST)
- net GND: now also TP23.1 (TEST), TP24.1 (TEST), TP25.1 (TEST), TP26.1 (TEST)
- net GP10: now also TP14.1 (TEST)
- net GP11: now also TP18.1 (TEST)
- net GP12: now also TP15.1 (TEST)
- net GP13: now also TP19.1 (TEST)
- net GP14: now also TP16.1 (TEST)
- net GP15: now also TP20.1 (TEST)
- net GP8: now also TP13.1 (TEST)
- net GP9: now also TP17.1 (TEST)
- net KBD_5V: now also TP6.1 (TEST)
- net KBD_CLOCK: now also TP10.1 (TEST)
- net KBD_DATA: now also TP9.1 (TEST)
- net MOUSE_5V: now also TP7.1 (TEST)
- net MOUSE_CLOCK: now also TP12.1 (TEST)
- net MOUSE_DATA: now also TP11.1 (TEST)
- net USB1_5V: now also TP4.1 (TEST)
- net USB1_FAULT: now also TP21.1 (TEST)
- net USB2_5V: now also TP5.1 (TEST)
- net USB2_FAULT: now also TP22.1 (TEST)
Other:
- note added: "8 / TEST ACCESS"
- note added: "Prototype: firmware and bench tests are required before use with the X16. See test-points.md and breadboard.md."
- note added: "Q = transistor. R = resistor. C = capacitor. U = chip. TP = test point. M1 numbers are carrier pins; use module GP labels."
- note added: "TP holes are optional probe contacts, not extra required parts. All GND test points are connected."
- note added: "USB data: probe existing R3.1 / R4.1 (keyboard D+ / D-) or R8.1 / R9.1 (mouse D+ / D-). No added USB stubs."
- note removed: "Prototype: firmware and bench tests are required before use with the X16. Cable wiring is in breadboard.md."
- note removed: "Q = transistor. R = resistor. C = capacitor. U = chip. M1 pin numbers are carrier numbers; use GP labels on the module."
